Commit message: Update gripper.urdf.xacro

File: gripper/urdf/gripper.urdf.xacro (robot description, xacro)
@@ -23,11 +23,11 @@
     <link name="gripper_base_link">
       <visual>
-        <geometry><box size="0.24 0.10 0.10"/></geometry>
+        <geometry><box size="0.24 0.08 0.08"/></geometry>
         <material name="gripper_grey"/>
       </visual>
       <collision>
-        <geometry><box size="0.24 0.10 0.10"/></geometry>
+        <geometry><box size="0.24 0.08 0.08"/></geometry>
       </collision>
-      <xacro:box_inertia m="1.0" w="0.24" h="0.10" d="0.10"/>
+      <xacro:box_inertia m="1.0" w="0.24" h="0.08" d="0.08"/>
     </link>
     <link name="right_finger">
